Commit message: VRX tunnel: calmer waves; RGL point cloud bridges + frame alignment; IMU frame relay; optional auto-forward with duration; YAML-driven launch and config; add tunnel_viz launch and docs

File: vrx_urdf/wamv_gazebo/urdf/components/wamv_rgl_lidar.xacro (robot description, xacro)
@@ -17,6 +17,8 @@
                                             plugin_filename:='RGLServerPluginInstance'
                                             plugin_name:='rgl::RGLServerPluginInstance'">
-    <!-- Derive default frame if not provided (use Pythonic ternary) -->
-    <xacro:property name="lidar_frame" value="${frame if frame else namespace + '/' + name + '_link'}"/>
+    <!-- Always bind the plugin frame to the actual link frame to ensure TF alignment.
+         Note: The optional 'frame' arg is ignored to avoid mismatches like
+         'front_lidar_link' vs the real link name 'RGLLidar_front_link'. -->
+    <xacro:property name="lidar_frame" value="${namespace + '/' + name + '_link'}"/>
     <!-- Define length variables for link positioning -->
     <xacro:property name="platform_z" value="${post_z_from}"/>

File: vrx_urdf/wamv_gazebo/urdf/wamv_gazebo.urdf.xacro (robot description, xacro)
@@ -75,6 +75,7 @@
     <plugin filename="libgz-sim-pose-publisher-system.so"
       name="gz::sim::systems::PosePublisher">
+      <!-- RobotStatePublisher already handles link frames; avoid noisy sensor entity frames. -->
       <publish_link_pose>false</publish_link_pose>
-      <publish_sensor_pose>true</publish_sensor_pose>
+      <publish_sensor_pose>false</publish_sensor_pose>
       <publish_collision_pose>false</publish_collision_pose>
       <publish_visual_pose>false</publish_visual_pose>
